File: Swallow-ethernet_memories.sch (KiCad schematic (older format))
At the start: 6 parts, among them P5 Ethernet_Slice, U8 S25FL064K, U9 DRAM-2MX16X4

Commit message: Converted LED resistors from individuals to array. Connected most signals.
Parts:
- removed W6: A10, TestPad-1mm, symbol TESTPOINT
Connections:
- wire segments 209 -> 204
Changed lines of the file:
@@
-EESchema Schematic File Version 2  date 01/10/2012 17:33:27
+EESchema Schematic File Version 2  date Mon 01 Oct 2012 22:14:03 BST
 LIBS:power
 LIBS:device
@@
 	6550 7250 6300 7250
 Wire Wire Line
-	10000 2250 10350 2250
-Wire Wire Line
 	7150 3450 7150 3400
 Wire Wire Line
@@
 	8450 1500 8950 1500
 Wire Wire Line
-	8950 1500 8950 1600
-Wire Wire Line
-	8950 1600 9000 1600
-Wire Wire Line
 	8450 1800 8750 1800
 Wire Wire Line
@@
 Wire Wire Line
 	9250 1400 8450 1400
-Wire Wire Line
-	10650 2950 10600 2950
-Wire Wire Line
-	10600 2950 10600 2850
 Connection ~ 10600 2850
 Wire Wire Line
@@
 B17 is unused INT_N\nB18 in unused RXER
 $Comp
-L +3.3V #PWR031
+L +3.3V #PWR033
 U 1 1 506889FB
 P 2200 3800
-F 0 "#PWR031" H 2200 3760 30  0001 C CNN
+F 0 "#PWR033" H 2200 3760 30  0001 C CNN
 F 1 "+3.3V" H 2200 3910 30  0000 C CNN
 	1    2200 3800
@@
 NoConn ~ 2900 5200
 $Comp
-L GND #PWR032
+L GND #PWR034
 U 1 1 506889D0
 P 2800 5300
-F 0 "#PWR032" H 2800 5300 30  0001 C CNN
+F 0 "#PWR034" H 2800 5300 30  0001 C CNN
 F 1 "GND" H 2800 5230 30  0001 C CNN
 	1    2800 5300
@@
 $EndComp
 $Comp
-L GND #PWR033
+L GND #PWR035
 U 1 1 506889CC
 P 3800 5300
-F 0 "#PWR033" H 3800 5300 30  0001 C CNN
+F 0 "#PWR035" H 3800 5300 30  0001 C CNN
 F 1 "GND" H 3800 5230 30  0001 C CNN
 	1    3800 5300
@@
 A9
 $Comp
-L +3.3V #PWR034
+L +3.3V #PWR036
 U 1 1 506882AB
 P 10300 2850
-F 0 "#PWR034" H 10300 2810 30  0001 C CNN
+F 0 "#PWR036" H 10300 2810 30  0001 C CNN
 F 1 "+3.3V" H 10300 2960 30  0000 C CNN
 	1    10300 2850
@@
 $EndComp
 $Comp
-L GND #PWR035
+L GND #PWR037
 U 1 1 4F5B70D6
 P 10400 2500
-F 0 "#PWR035" H 10400 2500 30  0001 C CNN
+F 0 "#PWR037" H 10400 2500 30  0001 C CNN
 F 1 "GND" H 10400 2430 30  0001 C CNN
 	1    10400 2500
 	1    0    0    -1
 $EndComp
-Text GLabel 10650 2950 2    60   Output ~ 0
-VDD_DRAM
 Text Label 6400 1750 0    60   ~ 0
 P4B0
@@
 DRAM_CLK
 $Comp
-L TESTPOINT W6
-U 1 1 4F622603
-P 9000 1450
-F 0 "W6" H 9000 1400 60  0000 C CNN
-F 1 "A10" H 9000 1450 20  0000 C CNN
-F 2 "TestPad-1mm" H 9000 1550 20  0001 C CNN
-	1    9000 1450
-	1    0    0    -1
-$EndComp
-$Comp
 L DRAM-4MX16X4 U9
 U 1 1 4F5A335A
@@
 D_CLK_EN
 $Comp
-L +3.3V #PWR036
+L +3.3V #PWR038
 U 1 1 4F5D0367
 P 9700 2500
-F 0 "#PWR036" H 9700 2460 30  0001 C CNN
+F 0 "#PWR038" H 9700 2460 30  0001 C CNN
 F 1 "+3.3V" H 9700 2610 30  0000 C CNN
 	1    9700 2500
@@
 VDD_Q
 $Comp
-L GND #PWR037
+L GND #PWR039
 U 1 1 4F5BE236
 P 7150 3450
-F 0 "#PWR037" H 7150 3450 30  0001 C CNN
+F 0 "#PWR039" H 7150 3450 30  0001 C CNN
 F 1 "GND" H 7150 3380 30  0001 C CNN
 	1    7150 3450
 	1    0    0    -1
 $EndComp
-Text Label 10150 2250 0    60   ~ 0
-VDD_DRAM
-Text GLabel 10000 2250 0    60   Output ~ 0
+Text Label 10750 2850 0    60   ~ 0
 VDD_DRAM
 Text HLabel 6550 6850 2    60   Output ~ 0
@@
 GPIO1
 $Comp
-L GND #PWR038
+L GND #PWR040
 U 1 1 4F5B6D20
 P 6850 6150
-F 0 "#PWR038" H 6850 6150 30  0001 C CNN
+F 0 "#PWR040" H 6850 6150 30  0001 C CNN
 F 1 "GND" H 6850 6080 30  0001 C CNN
 	1    6850 6150
@@
 $EndComp
 $Comp
-L +3.3V #PWR039
+L +3.3V #PWR041
 U 1 1 4F5B6D1D
 P 6650 6000
-F 0 "#PWR039" H 6650 5960 30  0001 C CNN
+F 0 "#PWR041" H 6650 5960 30  0001 C CNN
 F 1 "+3.3V" H 6650 6110 30  0000 C CNN
 	1    6650 6000
@@
 $EndComp
 $Comp
-L +3.3V #PWR040
+L +3.3V #PWR042
 U 1 1 4F5B6D0E
 P 8450 5650
-F 0 "#PWR040" H 8450 5610 30  0001 C CNN
+F 0 "#PWR042" H 8450 5610 30  0001 C CNN
 F 1 "+3.3V" H 8450 5760 30  0000 C CNN
 	1    8450 5650
@@
 BA1
 $Comp
-L GND #PWR041
+L GND #PWR043
 U 1 1 4F5B65E9
 P 7100 2350
-F 0 "#PWR041" H 7100 2350 30  0001 C CNN
+F 0 "#PWR043" H 7100 2350 30  0001 C CNN
 F 1 "GND" H 7100 2280 30  0001 C CNN
 	1    7100 2350
@@
 LDQM + UDQM = Output enable_N\nCan be used individually to set the device into 8bit mode.\n8 bit version of the device available.
 $Comp
-L GND #PWR042
+L GND #PWR044
 U 1 1 4F5B60D8
 P 7100 1000
-F 0 "#PWR042" H 7100 1000 30  0001 C CNN
+F 0 "#PWR044" H 7100 1000 30  0001 C CNN
 F 1 "GND" H 7100 930 30  0001 C CNN
 	1    7100 1000
@@
 $EndComp
 $Comp
-L GND #PWR043
+L GND #PWR045
 U 1 1 4F5B60D1
 P 8600 2500
-F 0 "#PWR043" H 8600 2500 30  0001 C CNN
+F 0 "#PWR045" H 8600 2500 30  0001 C CNN
 F 1 "GND" H 8600 2430 30  0001 C CNN
 	1    8600 2500
@@
 $EndComp
 $Comp
-L GND #PWR044
+L GND #PWR046
 U 1 1 4F5B60CC
 P 7100 2800
-F 0 "#PWR044" H 7100 2800 30  0001 C CNN
+F 0 "#PWR046" H 7100 2800 30  0001 C CNN
 F 1 "GND" H 7100 2730 30  0001 C CNN
 	1    7100 2800
@@
 $EndComp
 $Comp
-L GND #PWR045
+L GND #PWR047
 U 1 1 4F5B60C1
 P 8650 3100
-F 0 "#PWR045" H 8650 3100 30  0001 C CNN
+F 0 "#PWR047" H 8650 3100 30  0001 C CNN
 F 1 "GND" H 8650 3030 30  0001 C CNN
 	1    8650 3100
@@
 $EndComp
 $Comp
-L GND #PWR046
+L GND #PWR048
 U 1 1 4F5B5F9C
 P 7150 3650
-F 0 "#PWR046" H 7150 3650 30  0001 C CNN
+F 0 "#PWR048" H 7150 3650 30  0001 C CNN
 F 1 "GND" H 7150 3580 30  0001 C CNN
 	1    7150 3650

Commit message: Altered +5V capacitors to larger size for higher V rating. Changed reset chip cap from 100pF to 100nF to ensure a longer reset signal for the ethernet MAC.
Parts:
- added P8: PCIe_extra, symbol CONN_2
- added P9: RESET_N, symbol CONN_2
Connections:
- wire segments 204 -> 211
- no-connect marks 14 -> 12
