File: Swallow-ethernet_memories.sch (KiCad schematic (older format))
At the start: 7 parts, among them P5 Ethernet_Slice, P8 PCIe_extra, P9 RESET_N, U8 S25FL064K, U9 DRAM-2MX16X4

Commit message: Added proper GPIO header and connected a second GPIO to the flash part.
Connections:
- net labels added: MEM_LED
- wire segments 211 -> 213

Commit message: Added extra GPIO header from flash pins. Changed LED connection to CLK.
Connections:
- net labels added: GPIO3, L1_LED
- wire segments 213 -> 218
Changed lines of the file:
@@
-EESchema Schematic File Version 2  date Mon 08 Oct 2012 20:44:15 BST
+EESchema Schematic File Version 2  date Tue 09 Oct 2012 18:00:45 BST
 LIBS:power
 LIBS:device
@@
 $Descr A4 11700 8267
 encoding utf-8
-Sheet 3 4
+Sheet 2 4
 Title ""
-Date "8 oct 2012"
+Date "9 oct 2012"
 Rev ""
 Comp ""
@@
 $EndDescr
 Wire Wire Line
+	8650 6000 8650 5500
+Connection ~ 8450 6000
+Wire Wire Line
+	8650 6000 8450 6000
+Wire Wire Line
 	7750 5150 6400 5150
 Wire Wire Line
@@
 Wire Wire Line
 	6550 5250 7750 5250
+Wire Wire Line
+	6650 5750 6650 5400
+Connection ~ 6650 5750
+Wire Wire Line
+	6650 5400 7750 5400
+Wire Wire Line
+	8650 5500 8200 5500
+Text HLabel 8200 5500 0    60   BiDi ~ 0
+L1_LED
+Text HLabel 7750 5400 2    60   BiDi ~ 0
+GPIO3
 Text HLabel 7750 5000 2    60   Output ~ 0
 MEM_LED
 $Comp
-L GND #PWR042
+L GND #PWR027
 U 1 1 506AAE2B
 P 4000 6050
-F 0 "#PWR042" H 4000 6050 30  0001 C CNN
+F 0 "#PWR027" H 4000 6050 30  0001 C CNN
 F 1 "GND" H 4000 5980 30  0001 C CNN
 	1    4000 6050
@@
 B17 is unused INT_N\nB18 in unused RXER
 $Comp
-L +3.3V #PWR043
+L +3.3V #PWR028
 U 1 1 506889FB
 P 2200 3800
-F 0 "#PWR043" H 2200 3760 30  0001 C CNN
+F 0 "#PWR028" H 2200 3760 30  0001 C CNN
 F 1 "+3.3V" H 2200 3910 30  0000 C CNN
 	1    2200 3800
@@
 $EndComp
 $Comp
-L GND #PWR044
+L GND #PWR029
 U 1 1 506889D0
 P 2800 5300
-F 0 "#PWR044" H 2800 5300 30  0001 C CNN
+F 0 "#PWR029" H 2800 5300 30  0001 C CNN
 F 1 "GND" H 2800 5230 30  0001 C CNN
 	1    2800 5300
@@
 $EndComp
 $Comp
-L GND #PWR045
+L GND #PWR030
 U 1 1 506889CC
 P 3800 5300
-F 0 "#PWR045" H 3800 5300 30  0001 C CNN
+F 0 "#PWR030" H 3800 5300 30  0001 C CNN
 F 1 "GND" H 3800 5230 30  0001 C CNN
 	1    3800 5300
@@
 A9
 $Comp
-L +3.3V #PWR046
+L +3.3V #PWR031
 U 1 1 506882AB
 P 10300 2850
-F 0 "#PWR046" H 10300 2810 30  0001 C CNN
+F 0 "#PWR031" H 10300 2810 30  0001 C CNN
 F 1 "+3.3V" H 10300 2960 30  0000 C CNN
 	1    10300 2850
@@
 $EndComp
 $Comp
-L GND #PWR047
+L GND #PWR032
 U 1 1 4F5B70D6
 P 10400 2500
-F 0 "#PWR047" H 10400 2500 30  0001 C CNN
+F 0 "#PWR032" H 10400 2500 30  0001 C CNN
 F 1 "GND" H 10400 2430 30  0001 C CNN
 	1    10400 2500
@@
 D_CLK_EN
 $Comp
-L +3.3V #PWR048
+L +3.3V #PWR033
 U 1 1 4F5D0367
 P 9700 2500
-F 0 "#PWR048" H 9700 2460 30  0001 C CNN
+F 0 "#PWR033" H 9700 2460 30  0001 C CNN
 F 1 "+3.3V" H 9700 2610 30  0000 C CNN
 	1    9700 2500
@@
 VDD_Q
 $Comp
-L GND #PWR049
+L GND #PWR034
 U 1 1 4F5BE236
 P 7150 3450
-F 0 "#PWR049" H 7150 3450 30  0001 C CNN
+F 0 "#PWR034" H 7150 3450 30  0001 C CNN
 F 1 "GND" H 7150 3380 30  0001 C CNN
 	1    7150 3450
@@
 GPIO1
 $Comp
-L GND #PWR050
+L GND #PWR035
 U 1 1 4F5B6D20
 P 6850 6150
-F 0 "#PWR050" H 6850 6150 30  0001 C CNN
+F 0 "#PWR035" H 6850 6150 30  0001 C CNN
 F 1 "GND" H 6850 6080 30  0001 C CNN
 	1    6850 6150
@@
 $EndComp
 $Comp
-L +3.3V #PWR051
+L +3.3V #PWR036
 U 1 1 4F5B6D1D
 P 6650 6000
-F 0 "#PWR051" H 6650 5960 30  0001 C CNN
+F 0 "#PWR036" H 6650 5960 30  0001 C CNN
 F 1 "+3.3V" H 6650 6110 30  0000 C CNN
 	1    6650 6000
@@
 $EndComp
 $Comp
-L +3.3V #PWR052
+L +3.3V #PWR037
 U 1 1 4F5B6D0E
 P 8450 5650
-F 0 "#PWR052" H 8450 5610 30  0001 C CNN
+F 0 "#PWR037" H 8450 5610 30  0001 C CNN
 F 1 "+3.3V" H 8450 5760 30  0000 C CNN
 	1    8450 5650
@@
 BA1
 $Comp
-L GND #PWR053
+L GND #PWR038
 U 1 1 4F5B65E9
 P 7100 2350
-F 0 "#PWR053" H 7100 2350 30  0001 C CNN
+F 0 "#PWR038" H 7100 2350 30  0001 C CNN
 F 1 "GND" H 7100 2280 30  0001 C CNN
 	1    7100 2350
@@
 LDQM + UDQM = Output enable_N\nCan be used individually to set the device into 8bit mode.\n8 bit version of the device available.
 $Comp
-L GND #PWR054
+L GND #PWR039
 U 1 1 4F5B60D8
 P 7100 1000
-F 0 "#PWR054" H 7100 1000 30  0001 C CNN
+F 0 "#PWR039" H 7100 1000 30  0001 C CNN
 F 1 "GND" H 7100 930 30  0001 C CNN
 	1    7100 1000
@@
 $EndComp
 $Comp
-L GND #PWR055
+L GND #PWR040
 U 1 1 4F5B60D1
 P 8600 2500
-F 0 "#PWR055" H 8600 2500 30  0001 C CNN
+F 0 "#PWR040" H 8600 2500 30  0001 C CNN
 F 1 "GND" H 8600 2430 30  0001 C CNN
 	1    8600 2500
@@
 $EndComp
 $Comp
-L GND #PWR056
+L GND #PWR041
 U 1 1 4F5B60CC
 P 7100 2800
-F 0 "#PWR056" H 7100 2800 30  0001 C CNN
+F 0 "#PWR041" H 7100 2800 30  0001 C CNN
 F 1 "GND" H 7100 2730 30  0001 C CNN
 	1    7100 2800
@@
 $EndComp
 $Comp
-L GND #PWR057
+L GND #PWR042
 U 1 1 4F5B60C1
 P 8650 3100
-F 0 "#PWR057" H 8650 3100 30  0001 C CNN
+F 0 "#PWR042" H 8650 3100 30  0001 C CNN
 F 1 "GND" H 8650 3030 30  0001 C CNN
 	1    8650 3100
@@
 $EndComp
 $Comp
-L GND #PWR058
+L GND #PWR043
 U 1 1 4F5B5F9C
 P 7150 3650
-F 0 "#PWR058" H 7150 3650 30  0001 C CNN
+F 0 "#PWR043" H 7150 3650 30  0001 C CNN
 F 1 "GND" H 7150 3580 30  0001 C CNN
 	1    7150 3650

Commit message: Placed four 3mm mounting holes.
Parts:
- U8: value S25FL064K -> MX25L6445EM2I-10G
Changed lines of the file:
@@
-EESchema Schematic File Version 2  date Tue 09 Oct 2012 21:50:25 BST
+EESchema Schematic File Version 2  date Wed 10 Oct 2012 18:34:54 BST
 LIBS:power
 LIBS:device
@@
 Sheet 2 4
 Title ""
-Date "9 oct 2012"
+Date "10 oct 2012"
 Rev ""
 Comp ""
@@
 P 7650 5900
 F 0 "U8" H 7600 5650 60  0000 C CNN
-F 1 "S25FL064K" H 7600 6150 60  0000 C CNN
+F 1 "MX25L6445EM2I-10G" H 7600 6150 60  0000 C CNN
 F 2 "SO8NL" H 7600 6250 60  0001 C CNN
 	1    7650 5900

Commit message: Swapped BA0 & BA1 from 4 bit port to bits 13&14 of the address 16 bit port, following Andrew Stanford-Jason's suggestions. Re-laid out. GND plane also improved.
Connections:
- wire segments 218 -> 216
Changed lines of the file:
@@
-EESchema Schematic File Version 2  date Wed 10 Oct 2012 18:34:54 BST
+EESchema Schematic File Version 2  date Thu 11 Oct 2012 12:37:16 BST
 LIBS:power
 LIBS:device
@@
 Sheet 2 4
 Title ""
-Date "10 oct 2012"
+Date "11 oct 2012"
 Rev ""
 Comp ""
@@
 	8450 1700 8750 1700
 Wire Wire Line
-	6300 1950 6700 1950
-Wire Wire Line
 	7250 2100 6950 2100
 Wire Wire Line
@@
 Wire Wire Line
 	7100 2300 7250 2300
-Wire Wire Line
-	6300 2050 6700 2050
 Wire Wire Line
 	8450 1600 8750 1600
@@
 Text Label 8500 1700 0    60   ~ 0
 BA0
-Text Label 6550 1950 2    60   ~ 0
+Text Label 6850 3200 2    60   ~ 0
 BA0
-Text Label 6550 2050 2    60   ~ 0
+Text Label 6850 3300 2    60   ~ 0
 BA1
 $Comp

Commit message: Added clock buffer for L1 + ethernet MAC. Updated BOM.
Parts:
- added P16: P4B{2,3}, symbol CONN_2
Connections:
- net labels added: CLKA, CLKB, P4B2, P4B3
- net labels removed: CLK
- wire segments 216 -> 220
Changed lines of the file:
@@
-EESchema Schematic File Version 2  date Thu 11 Oct 2012 12:37:16 BST
+EESchema Schematic File Version 2  date Thu 11 Oct 2012 17:02:03 BST
 LIBS:power
 LIBS:device
@@
 Comment4 ""
 $EndDescr
+Text Label 6400 2050 0    60   ~ 0
+P4B3
+Text Label 6400 1950 0    60   ~ 0
+P4B2
+Wire Wire Line
+	6300 2050 6600 2050
+Wire Wire Line
+	9800 3450 9550 3450
 Wire Wire Line
 	8650 6000 8650 5500
@@
 Wire Wire Line
 	8650 5500 8200 5500
+Wire Wire Line
+	9800 3250 9550 3250
+Wire Wire Line
+	6300 1950 6600 1950
+Text Label 9600 3450 0    60   ~ 0
+P4B3
+Text Label 9600 3250 0    60   ~ 0
+P4B2
+$Comp
+L CONN_2 P16
+U 1 1 5076E89B
+P 10150 3350
+F 0 "P16" V 10100 3350 40  0000 C CNN
+F 1 "P4B{2,3}" V 10200 3350 40  0000 C CNN
+	1    10150 3350
+	1    0    0    -1
+$EndComp
 Text HLabel 8200 5500 0    60   BiDi ~ 0
 L1_LED
@@
 MEM_LED
 $Comp
-L GND #PWR027
+L GND #PWR34
 U 1 1 506AAE2B
 P 4000 6050
-F 0 "#PWR027" H 4000 6050 30  0001 C CNN
+F 0 "#PWR34" H 4000 6050 30  0001 C CNN
 F 1 "GND" H 4000 5980 30  0001 C CNN
 	1    4000 6050
@@
 B17 is unused INT_N\nB18 in unused RXER
 $Comp
-L +3.3V #PWR028
+L +3.3V #PWR31
 U 1 1 506889FB
 P 2200 3800
-F 0 "#PWR028" H 2200 3760 30  0001 C CNN
+F 0 "#PWR31" H 2200 3760 30  0001 C CNN
 F 1 "+3.3V" H 2200 3910 30  0000 C CNN
 	1    2200 3800
@@
 $EndComp
 $Comp
-L GND #PWR029
+L GND #PWR32
 U 1 1 506889D0
 P 2800 5300
-F 0 "#PWR029" H 2800 5300 30  0001 C CNN
+F 0 "#PWR32" H 2800 5300 30  0001 C CNN
 F 1 "GND" H 2800 5230 30  0001 C CNN
 	1    2800 5300
@@
 $EndComp
 $Comp
-L GND #PWR030
+L GND #PWR33
 U 1 1 506889CC
 P 3800 5300
-F 0 "#PWR030" H 3800 5300 30  0001 C CNN
+F 0 "#PWR33" H 3800 5300 30  0001 C CNN
 F 1 "GND" H 3800 5230 30  0001 C CNN
 	1    3800 5300
@@
 NoConn ~ 2900 3400
 Text GLabel 1900 4800 0    60   Input ~ 0
-CLK
+CLKB
 $Comp
 L CONN_PCIE-36 P5
@@
 A9
 $Comp
-L +3.3V #PWR031
+L +3.3V #PWR46
 U 1 1 506882AB
 P 10300 2850
-F 0 "#PWR031" H 10300 2810 30  0001 C CNN
+F 0 "#PWR46" H 10300 2810 30  0001 C CNN
 F 1 "+3.3V" H 10300 2960 30  0000 C CNN
 	1    10300 2850
@@
 $EndComp
 $Comp
-L GND #PWR032
+L GND #PWR47
 U 1 1 4F5B70D6
 P 10400 2500
-F 0 "#PWR032" H 10400 2500 30  0001 C CNN
+F 0 "#PWR47" H 10400 2500 30  0001 C CNN
 F 1 "GND" H 10400 2430 30  0001 C CNN
 	1    10400 2500
@@
 D_CLK_EN
 $Comp
-L +3.3V #PWR033
+L +3.3V #PWR45
 U 1 1 4F5D0367
 P 9700 2500
-F 0 "#PWR033" H 9700 2460 30  0001 C CNN
+F 0 "#PWR45" H 9700 2460 30  0001 C CNN
 F 1 "+3.3V" H 9700 2610 30  0000 C CNN
 	1    9700 2500
@@
 VDD_Q
 $Comp
-L GND #PWR034
+L GND #PWR40
 U 1 1 4F5BE236
 P 7150 3450
-F 0 "#PWR034" H 7150 3450 30  0001 C CNN
+F 0 "#PWR40" H 7150 3450 30  0001 C CNN
 F 1 "GND" H 7150 3380 30  0001 C CNN
 	1    7150 3450
@@
 RST_N
 Text GLabel 4150 7350 0    60   Input ~ 0
-CLK
+CLKA
 Text HLabel 4200 2650 0    60   Input ~ 0
 XLD4i
@@
 GPIO1
 $Comp
-L GND #PWR035
+L GND #PWR36
 U 1 1 4F5B6D20
 P 6850 6150
-F 0 "#PWR035" H 6850 6150 30  0001 C CNN
+F 0 "#PWR36" H 6850 6150 30  0001 C CNN
 F 1 "GND" H 6850 6080 30  0001 C CNN
 	1    6850 6150
@@
 $EndComp
 $Comp
-L +3.3V #PWR036
+L +3.3V #PWR35
 U 1 1 4F5B6D1D
 P 6650 6000
-F 0 "#PWR036" H 6650 5960 30  0001 C CNN
+F 0 "#PWR35" H 6650 5960 30  0001 C CNN
 F 1 "+3.3V" H 6650 6110 30  0000 C CNN
 	1    6650 6000
@@
 $EndComp
 $Comp
-L +3.3V #PWR037
+L +3.3V #PWR42
 U 1 1 4F5B6D0E
 P 8450 5650
-F 0 "#PWR037" H 8450 5610 30  0001 C CNN
+F 0 "#PWR42" H 8450 5610 30  0001 C CNN
 F 1 "+3.3V" H 8450 5760 30  0000 C CNN
 	1    8450 5650
@@
 BA1
 $Comp
-L GND #PWR038
+L GND #PWR38
 U 1 1 4F5B65E9
 P 7100 2350
-F 0 "#PWR038" H 7100 2350 30  0001 C CNN
+F 0 "#PWR38" H 7100 2350 30  0001 C CNN
 F 1 "GND" H 7100 2280 30  0001 C CNN
 	1    7100 2350
@@
 LDQM + UDQM = Output enable_N\nCan be used individually to set the device into 8bit mode.\n8 bit version of the device available.
 $Comp
-L GND #PWR039
+L GND #PWR37
 U 1 1 4F5B60D8
 P 7100 1000
-F 0 "#PWR039" H 7100 1000 30  0001 C CNN
+F 0 "#PWR37" H 7100 1000 30  0001 C CNN
 F 1 "GND" H 7100 930 30  0001 C CNN
 	1    7100 1000
@@
 $EndComp
 $Comp
-L GND #PWR040
+L GND #PWR43
 U 1 1 4F5B60D1
 P 8600 2500
-F 0 "#PWR040" H 8600 2500 30  0001 C CNN
+F 0 "#PWR43" H 8600 2500 30  0001 C CNN
 F 1 "GND" H 8600 2430 30  0001 C CNN
 	1    8600 2500
@@
 $EndComp
 $Comp
-L GND #PWR041
+L GND #PWR39
 U 1 1 4F5B60CC
 P 7100 2800
-F 0 "#PWR041" H 7100 2800 30  0001 C CNN
+F 0 "#PWR39" H 7100 2800 30  0001 C CNN
 F 1 "GND" H 7100 2730 30  0001 C CNN
 	1    7100 2800
@@
 $EndComp
 $Comp
-L GND #PWR042
+L GND #PWR44
 U 1 1 4F5B60C1
 P 8650 3100
-F 0 "#PWR042" H 8650 3100 30  0001 C CNN
+F 0 "#PWR44" H 8650 3100 30  0001 C CNN
 F 1 "GND" H 8650 3030 30  0001 C CNN
 	1    8650 3100
@@
 $EndComp
 $Comp
-L GND #PWR043
+L GND #PWR41
 U 1 1 4F5B5F9C
 P 7150 3650
-F 0 "#PWR043" H 7150 3650 30  0001 C CNN
+F 0 "#PWR41" H 7150 3650 30  0001 C CNN
 F 1 "GND" H 7150 3580 30  0001 C CNN
 	1    7150 3650
